Commit message: added diff cont and SLAM

File: description/lidar.xacro (robot description, xacro)
@@ -6,5 +6,5 @@
         <parent link = 'chassis'/>
         <child link = 'laser_frame'/>
-        <origin xyz="0.1 0 0.175" rpy='0 0 0'/>
+        <origin xyz="0.25 0.1 0.175" rpy='0 0 0'/>
     </joint>
     <link name='laser_frame'>
@@ -41,6 +41,6 @@
                 </scan>
                 <range>
-                    <min>0.3</min>
-                    <max>6</max>
+                    <min>0.15</min>
+                    <max>8</max>
                 </range>
             </ray>

File: description/robot.urdf.xacro (robot description, xacro)
@@ -10,4 +10,5 @@
     </xacro:unless>
     <!-- <xacro:include filename="gazebo_control.xacro"/> -->
+    <!-- <xacro:include filename="ros2_control.xacro"/> -->
     <xacro:include filename="lidar.xacro"/>
 </robot>

File: description/robot_core.xacro (robot description, xacro)
@@ -18,5 +18,14 @@
         <color rgba="1 0 0 1"/>
     </material>
+    <!-- Base Link -->
     <link name="base_link">
+    </link>
+    <!-- BASE_FOOTPRINT LINK -->
+    <joint name='base_footprint_joint' type='fixed'>
+        <parent link='base_link'/>
+        <child link='base_footprint'/>
+        <origin xyz='0 0 0' rpy='0 0 0'/>
+    </joint>
+    <link name="base_footprint">
     </link>
     <!-- CHASSIS LINK -->
@@ -40,5 +49,5 @@
             </geometry>
         </collision>
-        <xacro:inertial_box mass='0.5' x='0.3' y='0.3' z='0.15'>
+        <xacro:inertial_box mass='1.5' x='0.3' y='0.3' z='0.15'>
             <origin xyz="0.15 0 0.075" rpy="0 0 0"/>
         </xacro:inertial_box>

File: description/ros2_control.xacro (robot description, xacro)
@@ -1,57 +1,29 @@
 <?xml version="1.0"?>
 <robot xmlns:xacro="http://www.ros.org/wiki/xacro">
-    <!-- CHANGE PARAMETERS IF NEEDED -->
-    <ros2_control name="RealRobot" type="system">
-        <hardware>
-            <plugin>diffdrive_arduino/DiffDriveArduino</plugin>
-            <param name="left_wheel_name">left_wheel_joint</param>
-            <param name="right_wheel_name">right_wheel_joint</param>
-            <param name="loop_rate">30</param>
-            <param name="device">/dev/ttyUSB0</param>
-            <param name="baud_rate">57600</param>
-            <param name="timeout">1000</param>
-            <param name="enc_counts_per_rev">3436</param>
-        </hardware>
-        <joint name="left_wheel_joint">
-            <command_interface name="velocity">
-                <param name="min">-10</param>
-                <param name="max">10</param>
-            </command_interface>
-            <state_interface name="velocity"/>
-            <state_interface name="position"/>
-        </joint>
-        <joint name="right_wheel_joint">
-            <command_interface name="velocity">
-                <param name="min">-10</param>
-                <param name="max">10</param>
-            </command_interface>
-            <state_interface name="velocity"/>
-            <state_interface name="position"/>
-        </joint>
-    </ros2_control>
-    <!--     <ros2_control name="GazeboSystem" type="system">
+    <ros2_control name='GazeboSystem' type='system'>
         <hardware>
             <plugin>gazebo_ros2_control/GazeboSystem</plugin>
         </hardware>
-        <joint name="left_wheel_joint">
-            <command_interface name="velocity">
-                <param name="min">-10</param>
-                <param name="max">10</param>
+        <joint name='left_wheel_joint'>
+            <command_interface name='velocity'>
+                <param name='min'>-10</param>
+                <param name='max'>10</param>
+            <state_interface name='velocity'/>
             </command_interface>
-            <state_interface name="position" />
-            <state_interface name="velocity" />
+            <state_interface name='velocity'/>
+            <state_interface name='position'/>
         </joint>
-        <joint name="right_wheel_joint">
-            <command_interface name="velocity">
-                <param name="min">-10</param>
-                <param name="max">10</param>
+        <joint name='right_wheel_joint'>
+            <command_interface name='velocity'>
+                <param name='min'>-10</param>
+                <param name='max'>10</param>
             </command_interface>
-            <state_interface name="velocity" />
-            <state_interface name="position" />
+            <state_interface name='velocity'/>
+            <state_interface name='position'/>
         </joint>
-    </ros2_control>-->
+    </ros2_control>
     <gazebo>
-        <plugin filename="libgazebo_ros2_control.so" name="gazebo_ros2_control">
-            <parameters>/home/asak/dev_ws2/src/my_bot/config/my_controllers.ymal</parameters>
+        <plugin name='gazebo_ros2_control' filename='libgazebo_ros2_control.so'>
+            <parameters>$(find my_bot)/config/my_controllers.yaml</parameters>
         </plugin>
     </gazebo>
